File: RPi02W.kicad_sch (KiCad schematic)
At the start: 45 parts, among them J1 Raspberry_Pi_2_3, J3 AudioJack3_SwitchTR, J9 USB_C_Receptacle, SW1 SW_SPDT_MSM, SW10 SW_Push, SW11 SW_Push, SW12 SW_Push, SW13 SW_Push, SW14 SW_Push, SW2 SW_Push, SW3 SW_Push, SW4 SW_Push, SW5 SW_Push, SW6 SW_Push, SW7 SW_Push, SW8 SW_Push, SW9 SW_Push, U1 MCP73831-2-OT, U3 LM4861MX, U4 CR2013-MI2120

Commit message: Add files via upload
Other:
- note added: "EDITS: Cut trace between power switch and 5V line, making it only on/off. DD and DR gpio pins are swapped? FIXES NEEDED: Audio amplifier doesn't boost enough for external speaker, even with higher gain resistors"
- note removed: "MAKE SURE 3V3 WORKS HERE!"
- moved on the sheet: J9, U4
